Commit message: Change track joint type to continuous and update names

File: src/agro_robot_sim/urdf/sowbot_01.xacro (robot description, xacro)
@@ -104,8 +104,9 @@
       </inertial>
     </link>
-    <joint name="${prefix}_track_joint" type="fixed">
+    <joint name="${prefix}_track_joint" type="continuous">
       <parent link="base_link"/>
       <child  link="${prefix}_track_link"/>
       <origin xyz="0 ${y} 0" rpy="0 0 0"/>
+      <axis xyz="0 ${axis_y} 0"/>
     </joint>
     <!-- Drive roller (front) — full track height; forms the rounded front end -->
@@ -431,6 +432,6 @@
     <plugin filename="gz-sim-diff-drive-system"
             name="gz::sim::systems::DiffDrive">
-      <left_joint>left_drive_joint</left_joint>
-      <right_joint>right_drive_joint</right_joint>
+      <left_joint>left_track_joint</left_joint>
+      <right_joint>right_track_joint</right_joint>
       <wheel_separation>${track_sep}</wheel_separation>
       <wheel_radius>${drive_radius}</wheel_radius>
@@ -452,4 +453,6 @@
             name="gz::sim::systems::JointStatePublisher">
       <topic>joint_states</topic>
+      <joint_name>left_track_joint</joint_name>
+      <joint_name>right_track_joint</joint_name>
       <joint_name>left_drive_joint</joint_name>
       <joint_name>right_drive_joint</joint_name>

Commit message: Replace diff drive plugin with tracked vehicle plugin

File: src/agro_robot_sim/urdf/sowbot_01.xacro (robot description, xacro)
@@ -13,5 +13,5 @@
     OAK-D rear:       xyz="-0.438  0.273  0.951"
   Plugins (Gazebo Harmonic; topics bridged by ros_gz_bridge):
-    gz-sim-diff-drive-system       cmd_vel → /cmd_vel, odom → /odom  (skid-steer / track diff)
+    gz-sim-tracked-vehicle-system  cmd_vel → /cmd_vel, odom → /odom  (belt surface velocity)
     gz-sim-joint-state-publisher   joint_states → /joint_states
     gz-sim-sensors-system / imu-system / navsat-system
@@ -104,9 +104,8 @@
       </inertial>
     </link>
-    <joint name="${prefix}_track_joint" type="continuous">
+    <joint name="${prefix}_track_joint" type="fixed">
       <parent link="base_link"/>
       <child  link="${prefix}_track_link"/>
       <origin xyz="0 ${y} 0" rpy="0 0 0"/>
-      <axis xyz="0 ${axis_y} 0"/>
     </joint>
     <!-- Drive roller (front) — full track height; forms the rounded front end -->
@@ -424,24 +423,39 @@
     rpy="0 0.2618 ${pi}"/>
   <!-- ══════════════════════════════════════════════════════════════
-       DIFF DRIVE PLUGIN  (track skid-steer)
-       Left/right drive rollers are the powered joints.
-       wheel_separation = track_sep (centre-to-centre).
-       wheel_radius     = drive_radius.
-       ══════════════════════════════════════════════════════════════ -->
-  <gazebo>
-    <plugin filename="gz-sim-diff-drive-system"
-            name="gz::sim::systems::DiffDrive">
-      <left_joint>left_track_joint</left_joint>
-      <right_joint>right_track_joint</right_joint>
-      <wheel_separation>${track_sep}</wheel_separation>
-      <wheel_radius>${drive_radius}</wheel_radius>
-      <max_linear_acceleration>0.43</max_linear_acceleration>
-      <max_angular_acceleration>1.0</max_angular_acceleration>
-      <topic>cmd_vel</topic>
-      <odom_topic>odom</odom_topic>
-      <tf_topic>tf</tf_topic>
-      <odom_publish_frequency>50</odom_publish_frequency>
-      <frame_id>odom</frame_id>
-      <child_frame_id>base_footprint</child_frame_id>
+       TRACKED VEHICLE PLUGIN  (gz-sim8 / Harmonic)
+       TrackedVehicle handles cmd_vel → belt surface velocity.
+       TrackController per side sets the actual belt speed.
+       NOTE: TrackedVehicle does NOT publish odom/tf; use
+       ros_gz_bridge + a separate odometry node, or re-add
+       gz-sim-diff-drive-system in parallel for odom only
+       (with wheel_radius=${drive_radius}, joints=drive joints).
+       cmd_vel topic default: /model/amiga_ng/cmd_vel
+       ══════════════════════════════════════════════════════════════ -->
+  <gazebo>
+    <plugin filename="gz-sim-tracked-vehicle-system"
+            name="gz::sim::systems::TrackedVehicle">
+      <left_track><link>left_track_link</link></left_track>
+      <right_track><link>right_track_link</link></right_track>
+      <tracks_separation>${track_sep}</tracks_separation>
+      <tracks_height>${track_height}</tracks_height>
+      <steering_efficiency>0.5</steering_efficiency>
+    </plugin>
+  </gazebo>
+  <!-- TrackController: one per side; listens on
+       /model/amiga_ng/left_track_link/track_cmd_vel  (default) -->
+  <gazebo>
+    <plugin filename="gz-sim-track-controller-system"
+            name="gz::sim::systems::TrackController">
+      <link>left_track_link</link>
+      <min_velocity>-1.5</min_velocity>
+      <max_velocity>1.5</max_velocity>
+    </plugin>
+  </gazebo>
+  <gazebo>
+    <plugin filename="gz-sim-track-controller-system"
+            name="gz::sim::systems::TrackController">
+      <link>right_track_link</link>
+      <min_velocity>-1.5</min_velocity>
+      <max_velocity>1.5</max_velocity>
     </plugin>
   </gazebo>
@@ -453,6 +467,4 @@
             name="gz::sim::systems::JointStatePublisher">
       <topic>joint_states</topic>
-      <joint_name>left_track_joint</joint_name>
-      <joint_name>right_track_joint</joint_name>
       <joint_name>left_drive_joint</joint_name>
       <joint_name>right_drive_joint</joint_name>

Commit message: Add chassis inertia and update track height parameter
Added nominal chassis inertia to prevent ODE instability and updated track height parameter.

File: src/agro_robot_sim/urdf/sowbot_01.xacro (robot description, xacro)
@@ -64,4 +64,11 @@
       <material name="black"/>
     </visual>
+    <!-- Nominal chassis inertia; prevents ODE instability from a zero-mass parent
+         when all child links are fixed. Values approximate a 5 kg rigid frame
+         (pod/track inertias dominate; this just anchors the merged body). -->
+    <inertial>
+      <mass value="5.0"/>
+      <inertia ixx="0.5" ixy="0" ixz="0" iyy="1.0" iyz="0" izz="1.0"/>
+    </inertial>
   </link>
   <joint name="base_footprint_joint" type="fixed">
@@ -438,5 +445,5 @@
       <right_track><link>right_track_link</link></right_track>
       <tracks_separation>${track_sep}</tracks_separation>
-      <tracks_height>${track_height}</tracks_height>
+      <tracks_height>${drive_radius}</tracks_height>  <!-- half-height to contact surface, not full box height -->
       <steering_efficiency>0.5</steering_efficiency>
       <!-- Explicit global topic; without this the plugin defaults to

Commit message: Fix joint parent-child relationship in sowbot_01.xacro

File: src/agro_robot_sim/urdf/sowbot_01.xacro (robot description, xacro)
@@ -73,7 +73,7 @@
   </link>
   <joint name="base_footprint_joint" type="fixed">
-    <parent link="base_footprint"/>
-    <child  link="base_link"/>
-    <origin xyz="0 0 ${base_link_z}" rpy="0 0 0"/>
+    <parent link="base_link"/>
+    <child  link="base_footprint"/>
+    <origin xyz="0 0 -${base_link_z}" rpy="0 0 0"/>
   </joint>
   <!-- ══════════════════════════════════════════════════════════════

Commit message: Fix joint parent-child relationship and friction direction

File: src/agro_robot_sim/urdf/sowbot_01.xacro (robot description, xacro)
@@ -73,7 +73,7 @@
   </link>
   <joint name="base_footprint_joint" type="fixed">
-    <parent link="base_link"/>
-    <child  link="base_footprint"/>
-    <origin xyz="0 0 -${base_link_z}" rpy="0 0 0"/>
+    <parent link="base_footprint"/>
+    <child  link="base_link"/>
+    <origin xyz="0 0 ${base_link_z}" rpy="0 0 0"/>
   </joint>
   <!-- ══════════════════════════════════════════════════════════════
@@ -99,5 +99,5 @@
               <mu>2.0</mu>
               <mu2>2.0</mu2>
-              <fdir1>1 0 0</fdir1>
+              <fdir1>0 1 0</fdir1>
               <slip1>0.0</slip1>
               <slip2>0.0</slip2>
