Commit message: Add joint limits and dynamics to wheel joints

File: src/devkit_simulation/urdf/robo_caatinga.urdf.xacro (robot description, xacro)
@@ -218,4 +218,6 @@
       <origin xyz="${x} ${y} 0" rpy="0 0 0"/>
       <axis xyz="0 1 0"/>
+      <limit effort="100.0" velocity="10.0"/>
+      <dynamics damping="0.1" friction="0.1"/>
     </joint>
   </xacro:macro>

Commit message: Modify wheel inertia and add gazebo friction settings
Updated inertia values for the wheel and added gazebo friction parameters.

File: src/devkit_simulation/urdf/robo_caatinga.urdf.xacro (robot description, xacro)
@@ -196,21 +196,23 @@
         <origin xyz="0 0 0" rpy="${pi/2} 0 0"/>
         <geometry> <cylinder radius="${wheel_radius}" length="${wheel_width}"/> </geometry>
-        <surface>
-          <friction>
-            <ode>
-              <mu>1.5</mu>
-              <mu2>1.5</mu2>
-              <fdir1>1 0 0</fdir1>
-              <slip1>0.0</slip1>
-              <slip2>0.0</slip2>
-            </ode>
-          </friction>
-        </surface>
       </collision>
       <inertial>
         <mass value="10.0"/>
-        <inertia ixx="0.5" ixy="0" ixz="0" iyy="0.5" iyz="0" izz="0.5"/>
+        <!-- cylinder: ixx=iyy=(1/12)*m*(3r²+h²), izz=(1/2)*m*r² -->
+        <inertia ixx="0.156" ixy="0" ixz="0" iyy="0.156" iyz="0" izz="0.231"/>
       </inertial>
     </link>
+    <!-- Friction must be in <gazebo reference> for Harmonic — inline <surface>
+         inside URDF <collision> is silently dropped by sdformat conversion. -->
+    <gazebo reference="${prefix}_wheel">
+      <mu>1.5</mu>
+      <mu2>1.5</mu2>
+      <fdir1>1 0 0</fdir1>
+      <slip1>0.0</slip1>
+      <slip2>0.0</slip2>
+      <minDepth>0.001</minDepth>
+      <kp>1e6</kp>
+      <kd>1.0</kd>
+    </gazebo>
     <joint name="${prefix}_wheel_joint" type="continuous">
       <parent link="base_link"/>
