Commit message: Modify wheel friction and odometry settings
Updated friction parameters for better wheel traction and turning capability. Adjusted odometry settings to publish correct robot pose without drift.

File: src/devkit_simulation/urdf/ifarmate.urdf.xacro (robot description, xacro)
@@ -110,11 +110,22 @@
     </link>
     <!-- Friction in <gazebo reference> — inline <surface> in URDF
-         <collision> is dropped by sdformat conversion on Harmonic. -->
+         <collision> is dropped by sdformat conversion on Harmonic.
+         fdir1 (1 0 0, local X) is the rolling direction — mu/slip1 there
+         stay high-grip / zero-slip so the wheel doesn't spin out under
+         drive torque. mu2/slip2 govern the LATERAL axis (perpendicular to
+         fdir1) — this is the direction a diff-drive wheel must scrub
+         across during an in-place or skid turn. The original mu2=1.5,
+         slip2=0.0 gave the lateral axis the same zero-slip grip as the
+         rolling axis, which fights any lateral scrub and made the robot
+         effectively unable to turn (only drive forward/backward, where no
+         lateral scrub is needed). Lower mu2 and allow nonzero slip2 so
+         turning is kinematically possible while keeping rolling traction
+         (mu/slip1) unchanged. -->
     <gazebo reference="${prefix}_wheel">
       <mu>1.5</mu>
-      <mu2>1.5</mu2>
+      <mu2>0.3</mu2>
       <fdir1>1 0 0</fdir1>
       <slip1>0.0</slip1>
-      <slip2>0.0</slip2>
+      <slip2>0.3</slip2>
       <minDepth>0.001</minDepth>
       <kp>1e6</kp>
@@ -420,34 +431,9 @@
            not route (same fix as caatinga). -->
       <topic>/cmd_vel</topic>
-      <!-- DiffDrive DRIVES the robot but its integrated odom drifts under
-           wheel slip/blockage. Sink its odom+tf to unused topics; real
-           /odom + odom->base_footprint come from OdometryPublisher below
-           (ground-truth world pose). -->
-      <odom_topic>/_diffdrive_odom_unused</odom_topic>
-      <tf_topic>/_diffdrive_tf_unused</tf_topic>
+      <odom_topic>/odom</odom_topic>
+      <tf_topic>/tf</tf_topic>
       <odom_publish_frequency>50</odom_publish_frequency>
       <frame_id>odom</frame_id>
       <child_frame_id>base_footprint</child_frame_id>
-    </plugin>
-  </gazebo>
-  <!-- ══════════════════════════════════════════════════════════════
-       GROUND-TRUTH ODOMETRY (gz-sim8 / Harmonic)
-       Publishes /odom + odom->base_footprint from the model's REAL
-       simulator pose, so odom never drifts under wheel slip/blockage.
-       OdometryPublisher reports pose in the WORLD frame (verified: a
-       model spawned at (5,3) publishes odom (5,3), not 0). Gazebo world
-       == map/topo frame and map->odom is identity, so odom == the
-       robot's true map pose — drift-free, no EKF. Wire-compatible with
-       ros_gz_bridge.yaml (gz /odom + /tf).
-       ══════════════════════════════════════════════════════════════ -->
-  <gazebo>
-    <plugin filename="gz-sim-odometry-publisher-system"
-            name="gz::sim::systems::OdometryPublisher">
-      <odom_frame>odom</odom_frame>
-      <robot_base_frame>base_footprint</robot_base_frame>
-      <odom_topic>/odom</odom_topic>
-      <tf_topic>/tf</tf_topic>
-      <dimensions>3</dimensions>
-      <odom_publish_frequency>50</odom_publish_frequency>
     </plugin>
   </gazebo>

Commit message: odom + friction

File: src/devkit_simulation/urdf/ifarmate.urdf.xacro (robot description, xacro)
@@ -110,16 +110,5 @@
     </link>
     <!-- Friction in <gazebo reference> — inline <surface> in URDF
-         <collision> is dropped by sdformat conversion on Harmonic.
-         fdir1 (1 0 0, local X) is the rolling direction — mu/slip1 there
-         stay high-grip / zero-slip so the wheel doesn't spin out under
-         drive torque. mu2/slip2 govern the LATERAL axis (perpendicular to
-         fdir1) — this is the direction a diff-drive wheel must scrub
-         across during an in-place or skid turn. The original mu2=1.5,
-         slip2=0.0 gave the lateral axis the same zero-slip grip as the
-         rolling axis, which fights any lateral scrub and made the robot
-         effectively unable to turn (only drive forward/backward, where no
-         lateral scrub is needed). Lower mu2 and allow nonzero slip2 so
-         turning is kinematically possible while keeping rolling traction
-         (mu/slip1) unchanged. -->
+         <collision> is dropped by sdformat conversion on Harmonic. -->
     <gazebo reference="${prefix}_wheel">
       <mu>1.5</mu>
@@ -433,7 +422,34 @@
       <odom_topic>/odom</odom_topic>
       <tf_topic>/tf</tf_topic>
+      <!-- DiffDrive DRIVES the robot but its integrated odom drifts under
+           wheel slip/blockage. Sink its odom+tf to unused topics; real
+           /odom + odom->base_footprint come from OdometryPublisher below
+           (ground-truth world pose). -->
+      <odom_topic>/_diffdrive_odom_unused</odom_topic>
+      <tf_topic>/_diffdrive_tf_unused</tf_topic>
       <odom_publish_frequency>50</odom_publish_frequency>
       <frame_id>odom</frame_id>
       <child_frame_id>base_footprint</child_frame_id>
+    </plugin>
+  </gazebo>
+  <!-- ══════════════════════════════════════════════════════════════
+       GROUND-TRUTH ODOMETRY (gz-sim8 / Harmonic)
+       Publishes /odom + odom->base_footprint from the model's REAL
+       simulator pose, so odom never drifts under wheel slip/blockage.
+       OdometryPublisher reports pose in the WORLD frame (verified: a
+       model spawned at (5,3) publishes odom (5,3), not 0). Gazebo world
+       == map/topo frame and map->odom is identity, so odom == the
+       robot's true map pose — drift-free, no EKF. Wire-compatible with
+       ros_gz_bridge.yaml (gz /odom + /tf).
+       ══════════════════════════════════════════════════════════════ -->
+  <gazebo>
+    <plugin filename="gz-sim-odometry-publisher-system"
+            name="gz::sim::systems::OdometryPublisher">
+      <odom_frame>odom</odom_frame>
+      <robot_base_frame>base_footprint</robot_base_frame>
+      <odom_topic>/odom</odom_topic>
+      <tf_topic>/tf</tf_topic>
+      <dimensions>3</dimensions>
+      <odom_publish_frequency>50</odom_publish_frequency>
     </plugin>
   </gazebo>
