Commit message: Add inertial properties to ifarmate URDF

File: src/devkit_simulation/urdf/ifarmate.urdf.xacro (robot description, xacro)
@@ -369,4 +369,8 @@
       <material name="black"/>
     </visual>
+    <inertial>
+      <mass value="0.05"/>
+      <inertia ixx="0.0005" ixy="0" ixz="0" iyy="0.0005" iyz="0" izz="0.0005"/>
+    </inertial>
   </link>
   <joint name="imu_joint" type="fixed">

Commit message: Modify friction parameters in ifarmate.urdf.xacro
Updated friction parameters for gazebo reference in URDF.

File: src/devkit_simulation/urdf/ifarmate.urdf.xacro (robot description, xacro)
@@ -110,11 +110,16 @@
     </link>
     <!-- Friction in <gazebo reference> — inline <surface> in URDF
-         <collision> is dropped by sdformat conversion on Harmonic. -->
+         <collision> is dropped by sdformat conversion on Harmonic.
+         sdformat's urdf2sdf whitelist here is mu1/mu2/fdir1/minDepth/
+         kp/kd — NOT "mu". <mu> was silently falling through as an
+         unrecognized child of <link> (log: "XML Element[mu], child of
+         element[link], not defined in SDF") -> zero primary friction
+         on every wheel. slip1/slip2 are ODE-only params with no DART
+         equivalent (this world runs dartsim) and logged the same
+         warning for no effect — removed rather than faked. -->
     <gazebo reference="${prefix}_wheel">
-      <mu>2.0</mu>
+      <mu1>2.0</mu1>
       <mu2>0.3</mu2>
       <fdir1>1 0 0</fdir1>
-      <slip1>0.0</slip1>
-      <slip2>0.3</slip2>
       <minDepth>0.001</minDepth>
       <kp>1e6</kp>
