Commit message: Add camera link and joint to sowbot_01.xacro

File: src/devkit_simulation/urdf/sowbot_01.xacro (robot description, xacro)
@@ -430,4 +430,57 @@
     rpy="0 0.2618 ${pi}"/>
   <!-- ══════════════════════════════════════════════════════════════
+       ROW-FOLLOW CAMERA — identical to ifarmate.urdf.xacro's
+       camera_link/camera_sensor (same name, topic, FOV, tilt, and
+       absolute mount height above ground), so crop_row_params.yaml's
+       camera_height_m/camera_tilt_deg (1.055 m / -20 deg) and the
+       image_topic wiring apply unchanged on this platform too.
+       Mounted directly off base_link (not mast/pods), same rationale
+       as ifarmate: height spec holds regardless of other geometry.
+       base_link sits at base_link_z (=drive_radius) above ground here,
+       vs wheel_radius on ifarmate — z offset below is adjusted for
+       that so absolute height above ground still comes out to 1.055 m.
+       ══════════════════════════════════════════════════════════════ -->
+  <link name="camera_link">
+    <visual>
+      <origin xyz="0 0 0" rpy="0 0 0"/>
+      <geometry> <box size="0.03 0.09 0.03"/> </geometry>
+      <material name="black"/>
+    </visual>
+    <inertial>
+      <mass value="0.1"/>
+      <inertia ixx="0.001" ixy="0" ixz="0" iyy="0.001" iyz="0" izz="0.001"/>
+    </inertial>
+  </link>
+  <joint name="camera_joint" type="fixed">
+    <parent link="base_link"/>
+    <child  link="camera_link"/>
+    <origin xyz="${pod_len/2 - 0.02} 0 ${1.055 - base_link_z}" rpy="0 0 0"/>
+  </joint>
+  <!-- Gazebo camera sensor — publishes on /camera/image_raw (gz topic),
+       bridged to ROS via ros_gz_bridge.yaml. Pitched down 20° (rpy "0 0.35 0"),
+       same as ifarmate. use_camera:=false must be passed to neo.launch.py so
+       it subscribes to this topic rather than trying to open a V4L2 device. -->
+  <gazebo reference="camera_link">
+    <sensor name="camera_sensor" type="camera">
+      <always_on>true</always_on>
+      <update_rate>30</update_rate>
+      <topic>camera</topic>
+      <gz_frame_id>camera_link</gz_frame_id>
+      <pose>0 0 0 0 0.35 0</pose>
+      <camera>
+        <horizontal_fov>1.047</horizontal_fov>
+        <image>
+          <width>640</width>
+          <height>480</height>
+          <format>R8G8B8</format>
+        </image>
+        <clip>
+          <near>0.1</near>
+          <far>100</far>
+        </clip>
+      </camera>
+    </sensor>
+  </gazebo>
+  <!-- ══════════════════════════════════════════════════════════════
        TRACKED VEHICLE PLUGIN  (gz-sim8 / Harmonic)
        TrackedVehicle handles cmd_vel → belt surface velocity.

Commit message: Add gazebo friction settings for track links
Added gazebo friction parameters for left and right tracks to ensure proper ground interaction during simulation.

File: src/devkit_simulation/urdf/sowbot_01.xacro (robot description, xacro)
@@ -159,4 +159,18 @@
   <xacro:track prefix="left"  y=" ${track_half}" axis_y=" 1"/>
   <xacro:track prefix="right" y="-${track_half}" axis_y="-1"/>
+  <!-- Native <collision><surface><friction> above is silently dropped on
+       URDF->SDF conversion (Gazebo Harmonic) — without this, tracks have
+       zero ground friction and spin in place. This is the form that
+       actually survives conversion. -->
+  <gazebo reference="left_track_link">
+    <mu1>0.7</mu1>
+    <mu2>150</mu2>
+    <fdir1>0 1 0</fdir1>
+  </gazebo>
+  <gazebo reference="right_track_link">
+    <mu1>0.7</mu1>
+    <mu2>150</mu2>
+    <fdir1>0 1 0</fdir1>
+  </gazebo>
   <!-- ══════════════════════════════════════════════════════════════
        SIDE BODY PODS  (two boxes above the tracks — the split body)
@@ -530,11 +544,13 @@
        joint velocities into odometry, matching the unscoped /odom
        gz topic that ros_gz_bridge.yaml expects.
-       TF: deliberately NOT publishing tf_topic here. fusioncore is
-       the sole publisher of odom->base_link (fed by bridged
-       /gnss/fix, /imu/data, /odom/wheels — the latter is this
-       plugin's /odom topic, relayed). Ground-truth /odom stays
-       available as a plain topic for error analysis / RTK-outage
-       testing; it just doesn't touch TF anymore. Two odom->base_link
-       broadcasters (this + fusioncore) would silently race.
+       TF: publish_tf explicitly false. fusioncore is the sole
+       publisher of odom->base_link (fed by bridged /gnss/fix,
+       /imu/data, /odom/wheels — the latter is this plugin's /odom
+       topic, relayed). Ground-truth /odom stays available as a
+       plain topic for error analysis / RTK-outage testing; it just
+       doesn't touch TF anymore. Two odom->base_link broadcasters
+       (this + fusioncore) would silently race — omitting tf_topic
+       alone does NOT prevent this; the plugin still broadcasts on
+       its default TF topic unless publish_tf is set false here.
        ══════════════════════════════════════════════════════════════ -->
   <gazebo>
@@ -551,4 +567,5 @@
       <child_frame_id>base_link</child_frame_id>
       <odom_publish_frequency>50</odom_publish_frequency>
+      <publish_tf>false</publish_tf>
     </plugin>
   </gazebo>

Commit message: fix: change track joints to continuous and fix TrackedVehicle plugin params

File: src/devkit_simulation/urdf/sowbot_01.xacro (robot description, xacro)
@@ -84,5 +84,5 @@
        ══════════════════════════════════════════════════════════════ -->
   <xacro:macro name="track" params="prefix y axis_y">
-    <!-- Belt body (visual + collision); fixed to base_link -->
+    <!-- Belt body (visual + collision) -->
     <link name="${prefix}_track_link">
       <visual>
@@ -111,8 +111,9 @@
       </inertial>
     </link>
-    <joint name="${prefix}_track_joint" type="fixed">
+    <joint name="${prefix}_track_joint" type="continuous">
       <parent link="base_link"/>
       <child  link="${prefix}_track_link"/>
       <origin xyz="0 ${y} 0" rpy="0 0 0"/>
+      <axis xyz="0 ${axis_y} 0"/>
     </joint>
     <!-- Drive roller (front) — full track height; forms the rounded front end -->
@@ -524,17 +525,6 @@
       <right_track><link>right_track_link</link></right_track>
       <tracks_separation>${track_sep}</tracks_separation>
-      <!-- Was <tracks_height> (typo'd, silently dropped/defaulted by
-           the plugin's LoadParam fallback). Correct element name per
-           the gz-sim TrackedVehicle schema is singular "track_height". -->
-      <track_height>${drive_radius}</track_height>  <!-- half-height to contact surface, not full box height -->
+      <tracks_height>${drive_radius}</tracks_height>
       <steering_efficiency>0.5</steering_efficiency>
-      <!-- Vehicle-level speed limit. min_velocity/max_velocity are NOT
-           TrackController parameters (they were previously placed there
-           and silently ignored) — they belong here, under
-           TrackedVehicle's <linear_velocity>. -->
-      <linear_velocity>
-        <min_velocity>-1.5</min_velocity>
-        <max_velocity>1.5</max_velocity>
-      </linear_velocity>
       <!-- Explicit global topic; without this the plugin defaults to
            /model/{entity_name}/cmd_vel which the bridge does not route. -->
@@ -548,4 +538,6 @@
             name="gz::sim::systems::TrackController">
       <link>left_track_link</link>
+      <min_velocity>-1.5</min_velocity>
+      <max_velocity>1.5</max_velocity>
     </plugin>
   </gazebo>
@@ -554,4 +546,6 @@
             name="gz::sim::systems::TrackController">
       <link>right_track_link</link>
+      <min_velocity>-1.5</min_velocity>
+      <max_velocity>1.5</max_velocity>
     </plugin>
   </gazebo>
@@ -580,5 +574,4 @@
       <wheel_separation>${track_sep}</wheel_separation>
       <wheel_radius>${drive_radius}</wheel_radius>
-      <!-- unused sink topic: never publish real cmd_vel here -->
       <topic>_unused_diffdrive_cmd_vel</topic>
       <odom_topic>odom</odom_topic>

Commit message: fix: keep sowbot tracks fixed to chassis so TrackedVehicle drives it
gz-sim's TrackedVehicle/TrackController drive the robot by a moving contact
surface on the belt's ground patch (conveyor effect), not by rotating a belt
joint. Fixing the belt to base_link also removes the free pivot at the axle
that let the chassis rock like an inverted pendulum. preserveFixedJoint
keeps left/right_track_link as real links (URDF->SDF lumps fixed-joint
children into the parent by default, so TrackController could never find
them). Verified: with this the sowbot drives and turns level.

File: src/devkit_simulation/urdf/sowbot_01.xacro (robot description, xacro)
@@ -84,5 +84,11 @@
        ══════════════════════════════════════════════════════════════ -->
   <xacro:macro name="track" params="prefix y axis_y">
-    <!-- Belt body (visual + collision) -->
+    <!-- Belt body (visual + collision). FIXED to base_link: gz-sim's
+         TrackedVehicle/TrackController drive the robot by setting a moving
+         contact surface on the belt's ground patch (conveyor effect), NOT by
+         rotating a belt joint — see gz-sim tracked_vehicle_simple.sdf (track
+         joints are type='fixed' there). Keeping the belt fixed to the chassis
+         also removes the free pivot at the belt axle that let the chassis
+         rock like an inverted pendulum and lose balance. -->
     <link name="${prefix}_track_link">
       <visual>
@@ -111,9 +117,8 @@
       </inertial>
     </link>
-    <joint name="${prefix}_track_joint" type="continuous">
+    <joint name="${prefix}_track_joint" type="fixed">
       <parent link="base_link"/>
       <child  link="${prefix}_track_link"/>
       <origin xyz="0 ${y} 0" rpy="0 0 0"/>
-      <axis xyz="0 ${axis_y} 0"/>
     </joint>
     <!-- Drive roller (front) — full track height; forms the rounded front end -->
@@ -160,4 +165,17 @@
   <xacro:track prefix="left"  y=" ${track_half}" axis_y=" 1"/>
   <xacro:track prefix="right" y="-${track_half}" axis_y="-1"/>
+  <!-- sdformat's URDF->SDF conversion lumps every fixed joint's child link
+       into its parent by default, so left/right_track_link would silently
+       disappear and TrackController could never find them (gzwarn + return;
+       robot never moves). preserveFixedJoint keeps these two as real links.
+       Verified in sim (2026-08-08): with this tag the sowbot drives and turns
+       level; without it, TrackedVehicle publishes belt cmds but the robot
+       stays put. -->
+  <gazebo reference="left_track_joint">
+    <preserveFixedJoint>true</preserveFixedJoint>
+  </gazebo>
+  <gazebo reference="right_track_joint">
+    <preserveFixedJoint>true</preserveFixedJoint>
+  </gazebo>
   <!-- Native <collision><surface><friction> above is silently dropped on
        URDF->SDF conversion (Gazebo Harmonic) — without this, tracks have
